File: CanLite.kicad_pcb (KiCad board)
At the start: 2 copper layers, 40 x 53.6 mm, 42 parts, among them J1 Conn_01x06, J2 Conn_01x03, J3 CAN, J4 12V, U1 ESP32-WROOM-32D, U2 VN750PS-E, U3 VN750PS-E, U4 SN65HVD231, U5 LMR14006

Commit message: Released rev.D
Parts:
- removed the R10 at (124.4, 82.2)
- removed R13: 10K, Resistor_SMD:R_0603_1608Metric
- removed the R6 at (117.4, 82.2)
- removed the R7 at (115.8, 82.2)
- removed the R9 at (126.0, 82.2)
- removed the U2 at (117.4, 88.6)
- removed the U3 at (124.4, 88.6)
- added R8: 10K, Resistor_SMD:R_0603_1608Metric, F.Cu at (124.8, 78.0)
- added TP3: IO25, TestPoint:TestPoint_Pad_D1.0mm, F.Cu at (109.2, 64.2)
- added TP4: IO26, TestPoint:TestPoint_Pad_D1.0mm, F.Cu at (111.0, 65.5)
- added TP5: IO27, TestPoint:TestPoint_Pad_D1.0mm, F.Cu at (109.2, 66.8)
- added TP6: IO32, TestPoint:TestPoint_Pad_D1.0mm, F.Cu at (109.2, 61.8)
- added U4: BTS452T, Package_TO_SOT_SMD:TO-252-4, F.Cu at (117.8, 87.2)
- added U5: BTS452T, Package_TO_SOT_SMD:TO-252-4, F.Cu at (127.0, 87.2)
- J3: renamed from J1; value Conn_01x06 -> VOLTLINK
- L1: footprint Voltlog:Inductor_7.5x6.6 -> voltlog:Inductor_7.5x6.6
- moved JP1 10.5 mm to (138.4, 85.9), turned to 90 degrees
- moved R7 5.80 mm to (123.0, 78.0)
- moved D3 3.26 mm to (123.0, 74.8)
- moved V1 3.11 mm to (104.5, 69.0)
- moved R4 2.00 mm to (124.8, 74.8), turned to 270 degrees
- moved J2 1.20 mm to (131.9, 99.6)
- moved J1 1.08 mm to (106.7, 99.6)
- moved R1 0.25 mm to (109.2, 59.0)
- moved L1 0.20 mm to (110.5, 77.0)
- renumbered C6 to C1, C7 to C2, C8 to C3, C3 to C4, C1 to C5, C2 to C6, C5 to C7, C4 to C8, D3 to D1, D4 to D2, D1 to D3, D2 to D4, J4 to J1, J3 to J2, J2 to J4, R4 to R10, R11 to R2, R14 to R3, R2 to R4, R12 to R5, R8 to R6, R5 to R7, R3 to R9, TP2 to TP1, TP3 to TP2, TP1 to TP7, U5 to U1, U1 to U2, U4 to U3
Connections:
- U2 pad 10: Net-(U1-Pad10) -> /IO25
- U2 pad 11: Net-(U1-Pad11) -> /IO26
- U2 pad 12: Net-(U1-Pad12) -> /IO27
- U2 pad 27: /STATUS1 -> Net-(U2-Pad27)
- U2 pad 30: /STATUS2 -> Net-(U2-Pad30)
- U2 pad 8: Net-(U1-Pad8) -> /IO32
Routing:
- net /STATUS2: track 27.6 -> 0.00 mm, vias 2 -> 0
- net /STATUS1: track 24.8 -> 0.00 mm
- net Net-(R8-Pad1): track 0.00 -> 17.7 mm, vias 0 -> 2
- net Net-(R7-Pad1): track 3.44 -> 21.1 mm, vias 0 -> 2
- net +3V3: track 103.1 -> 89.0 mm, vias 0 -> 2
- net /OUT1: track 0.00 -> 9.44 mm
- net /OUT2: track 0.00 -> 9.06 mm
- net Net-(JP1-Pad1): track 10.5 -> 1.97 mm
- net /CAN_L: track 14.3 -> 19.3 mm
- net Net-(R6-Pad1) (its old number): track 4.90 -> 0.00 mm
- net Net-(R10-Pad1): track 4.90 -> 0.00 mm
- net /CTRL2: track 27.9 -> 23.2 mm
- net /IO32: track 0.00 -> 4.30 mm
- net /IO25: track 0.00 -> 4.28 mm
- net /IO27: track 0.00 -> 4.26 mm
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- added copper zone on F.Cu, net +3V3
Other:
- board text added: "4021"
- board text added: "IO25"
- board text added: "IO26"
- board text added: "IO27"
- board text added: "IO32"
- board text added: "revD"
- board text removed: "0421"
- board text removed: "revB"
