File: CanLite.sch (KiCad schematic (older format))
At the start: 42 parts, among them J1 VOLTLINK, J2 Conn_01x03, J3 CAN, J4 12V, U1 ESP32-WROOM-32D, U2 VN750PS-E, U3 VN750PS-E, U4 SN65HVD231, U5 LMR14006

Commit message: Released rev.D
Parts:
- removed R10, R13, R6, R7, R9: 10K, Resistor_SMD:R_0603_1608Metric, symbol Device:R_US
- removed U2, U3: VN750PS-E, Package_SO:SO-8_3.9x4.9mm_P1.27mm, symbol voltlog:VN750PS-E
- added R8: 10K, Resistor_SMD:R_0603_1608Metric, symbol Device:R_US
- added TP3: IO25, TestPoint:TestPoint_Pad_D1.0mm, symbol Connector:TestPoint_Alt
- added TP4: IO26, TestPoint:TestPoint_Pad_D1.0mm, symbol Connector:TestPoint_Alt
- added TP5: IO27, TestPoint:TestPoint_Pad_D1.0mm, symbol Connector:TestPoint_Alt
- added TP6: IO32, TestPoint:TestPoint_Pad_D1.0mm, symbol Connector:TestPoint_Alt
- added U4, U5: BTS452T, Package_TO_SOT_SMD:TO-252-4, symbol voltlog:BTS452T
- L1: footprint Voltlog:Inductor_7.5x6.6 -> voltlog:Inductor_7.5x6.6; LCSC C341775 -> C436550; PN LQH3NPN2R2MJRL -> PSPMAA0603-8R2M-ANF
- renumbered C6 to C1, C7 to C2, C8 to C3, C3 to C4, C1 to C5, C2 to C6, C5 to C7, C4 to C8, D3 to D1, D4 to D2, D1 to D3, D2 to D4, J4 to J1, J3 to J2, J1 to J3, J2 to J4, R4 to R10, R11 to R2, R14 to R3, R2 to R4, R12 to R5, R8 to R6, R5 to R7, R3 to R9, TP2 to TP1, TP3 to TP2, TP1 to TP7, U5 to U1, U1 to U2, U4 to U3
Connections:
- net +BATT: now also U4.3 (Vbb), U5.3 (Vbb)
- net CTRL2: now also R8.2
- net GND: now also U4.1 (GND), U5.1 (GND)
- net OUT1: now also U4.5 (OUT)
- net OUT2: now also U5.5 (OUT)
- net at R7.1: now also U4.2 (IN)
- net IO25: now reaches U2.10 (IO25)
- net IO25: now also TP3.1
- net IO26: now reaches U2.11 (IO26)
- net IO26: now also TP4.1
- net IO27: now reaches U2.12 (IO27)
- net IO27: now also TP5.1
- net IO32: now reaches U2.8 (IO32)
- net IO32: now also TP6.1
- net STATUS1: no longer names the net of U2.27 (IO16)
- net STATUS2: no longer names the net of U2.30 (IO18)
- new net: R8.1, U5.2 (IN)
